Commit message: V56: shift rivet zone +0.30m east, remove cabin keep indicator, J5=-90 natural
- world_to_riveting_zone moved from (0.692, 1.259, 1.000) to (0.992, ...)
  so the cobot reaches LOAD seat with joint5 = -pi/2 as the natural IK
  solution (verified via scripts/probe_j5_reach.py).
- Riveting cabin (posts/canopy/lip/tray/back wall) removed.  Only the
  stack-light indicator (post + red/amber/green lamps) survives,
  mounted directly on the new riveting_zone.  The disc + fixtures +
  pistons + sensor are untouched (they parent to riveting_zone).
- resolve_poses.py: new RIVETING_ZONE_DX_SHIFT = 0.300 constant; J5
  hard-locked to -pi/2 after every IK call in the LOAD_RIVET branch
  (seeds also biased to J5=-pi/2); scoring now orders by j5_err first.
- resolved_poses.py regenerated: all 7 LOAD/RIVET poses land J5 at
  -1.570796 (-90.0000 deg) exactly; PLACE_LOAD FK error 0.16 mm.
- object_manager DISC_CENTER_X moved 0.677 -> 0.977 to track the new
  fixture XY (fallback path only; TF lookups are authoritative).
- New v56_geom_test.py verifies J5 = -90 deg on every LOAD/RIVET pose
  and the FK CAFI XYZ lies within 25 mm of the URDF seat.

Co-Authored-By: Claude Opus 4.7 (1M context) <noreply@anthropic.com>

File: src/schneider_cell_description/urdf/schneider_cell.urdf.xacro (robot description, xacro)
@@ -416,36 +416,78 @@
                     height="0.150" wall_t="0.005"
                     bottom_z="1.000" material="bin_reject"/>
-  <!-- ===== V37 Riveting zone anchor (disc CENTRE on mesa top) =========
-       Anchored at world (0.692, 1.259, 1.000) per DXF disco position.
-       The disc itself is mounted on this anchor; the cabin overhead
-       sits NORTH of the disc to clear the cobot working area.        -->
+  <!-- ===== V56 Riveting zone anchor (disc CENTRE on mesa top) =========
+       V56 shifts the disc eastward by +0.300 m so the cobot can reach
+       the LOAD seat with joint5 = -pi/2 (= -90 deg) — the IK probe
+       under scripts/probe_j5_reach.py shows convergent J5=-90
+       solutions in the [0.25, 0.40] m range; +0.30 m is the smallest
+       shift that keeps every joint comfortably inside its limit while
+       leaving > 50 mm clearance between the disc rim and the cobot
+       pedestal.
+         old anchor: world (0.692, 1.259, 1.000)
+         new anchor: world (0.992, 1.259, 1.000)         -->
   <link name="riveting_zone"/>
   <joint name="world_to_riveting_zone" type="fixed">
     <parent link="world"/>
     <child  link="riveting_zone"/>
-    <origin xyz="0.692 1.259 1.000" rpy="0 0 0"/>
+    <origin xyz="0.992 1.259 1.000" rpy="0 0 0"/>
   </joint>
-  <!-- V44 cabin: SHRUNK to give the cobot clean entry from the south.
-       V43 had cabin_size 0.700x0.400 with canopy at z=1.500.  V44
-       reduces footprint to 0.450x0.300 and height to 0.350 (canopy at
-       world z=1.350).  Canopy footprint extends NORTH of the disc only
-       (press_offset_y still 0.200 m), so the cobot approach corridor
-       to LOAD (from the south) is now completely open.
-         old cabin Y span at LOAD (y=1.109): 1.259 + 0.200 +/- 0.200 = [1.259, 1.659]
-         new cabin Y span at LOAD (y=1.109): 1.259 + 0.200 +/- 0.150 = [1.309, 1.609]
-       The new south edge of the canopy is at y=1.309 — 200 mm NORTH
-       of the LOAD seat (y=1.109).  The cobot wrist no longer collides
-       with the canopy during APPROACH_LOAD / RELEASE_LOAD / PICK_RIVETED.
-       Canopy top at z=1.350 clears CAFI top (z=1.136) by 214 mm.    -->
-  <xacro:riveting_station_features name="rivet_station"
-                                   parent="riveting_zone"
-                                   zone_size_x="0.500"
-                                   zone_size_y="0.350"
-                                   cabin_size_x="0.450"
-                                   cabin_size_y="0.300"
-                                   cabin_height="0.350"
-                                   press_offset_x="0"
-                                   press_offset_y="0.200"
-                                   include_press="false"/>
+  <!-- V56 RIVETING INDICATOR (cabin removed).
+       The user asked to drop the full riveting cabin (posts + canopy
+       + lip + tray + back wall) and keep ONLY the visual indicator
+       that signals whether riveting is in progress.  We replace the
+       whole `riveting_station_features` macro with a small stack
+       light mounted directly on the mesa next to the disc.  The
+       three lamp spheres mirror the V54 cabin lamps (red / amber /
+       green) and remain a static visual cue — the functional state
+       is the /rivet/active topic, already surfaced on the HMI as
+       DO3 Remachado.  -->
+  <link name="rivet_indicator_post">
+    <visual>
+      <origin xyz="0 0 0" rpy="0 0 0"/>
+      <geometry><cylinder radius="0.012" length="0.300"/></geometry>
+      <material name="station_pillar"/>
+    </visual>
+  </link>
+  <joint name="riveting_zone_to_indicator_post" type="fixed">
+    <parent link="riveting_zone"/>
+    <child  link="rivet_indicator_post"/>
+    <origin xyz="-0.220 0.000 0.150" rpy="0 0 0"/>
+  </joint>
+  <link name="rivet_indicator_lamp_red">
+    <visual>
+      <origin xyz="0 0 0" rpy="0 0 0"/>
+      <geometry><sphere radius="0.025"/></geometry>
+      <material name="lamp_red"/>
+    </visual>
+  </link>
+  <joint name="indicator_post_to_lamp_red" type="fixed">
+    <parent link="rivet_indicator_post"/>
+    <child  link="rivet_indicator_lamp_red"/>
+    <origin xyz="0 0 0.180" rpy="0 0 0"/>
+  </joint>
+  <link name="rivet_indicator_lamp_amber">
+    <visual>
+      <origin xyz="0 0 0" rpy="0 0 0"/>
+      <geometry><sphere radius="0.025"/></geometry>
+      <material name="lamp_amber"/>
+    </visual>
+  </link>
+  <joint name="indicator_post_to_lamp_amber" type="fixed">
+    <parent link="rivet_indicator_post"/>
+    <child  link="rivet_indicator_lamp_amber"/>
+    <origin xyz="0 0 0.130" rpy="0 0 0"/>
+  </joint>
+  <link name="rivet_indicator_lamp_green">
+    <visual>
+      <origin xyz="0 0 0" rpy="0 0 0"/>
+      <geometry><sphere radius="0.025"/></geometry>
+      <material name="lamp_green"/>
+    </visual>
+  </link>
+  <joint name="indicator_post_to_lamp_green" type="fixed">
+    <parent link="rivet_indicator_post"/>
+    <child  link="rivet_indicator_lamp_green"/>
+    <origin xyz="0 0 0.080" rpy="0 0 0"/>
+  </joint>
   <!-- ===== V52 Turntable rivet cell (drop-in from user's package) =======
        The whole rivet station (rotating disc, NEMA + base, belt, two

Commit message: V57: shift conveyor +30cm, lock J6 PICK=LOAD, 3cm safety margin
- Conveyor + suministro + sensor_conveyor_end + conveyor_drive_motor
  shifted +0.300 m EAST.  Pick at world X=1.535 (was 1.235); SPAWN at
  X=1.920 (was 1.620).  All inside mesa (x in [0.442, 2.062]).
- resolve_poses: J6 hard-locked to J6_PICK_CONVEYOR across the LOAD/
  RIVET group (APPROACH, PLACE, RELEASE, RETREAT, PICK_RIVETED, LIFT).
  Wrist no longer rolls during the carry — CAFI stays visually still.
  All 7 LOAD/RIVET poses land J6 = -2.373404 rad (delta < 0.001 mrad).
- conveyor_sim + object_manager X constants updated to match.
- New v57_collision_test.py: 17 world AABB/cylinder obstacles, samples
  every pose AND 10 interp steps per trajectory segment, fails if any
  cobot link comes within 3 cm.  Grasp center excluded (virtual TCP,
  not a physical link).

Tests (all PASS):
 - v57_collision_test: 0 violations across 19 poses + 27 segments
 - v55_aggressive_test: 52 CAFIs throughput + START/STOP/RESET cycle
 - v56_geom_test: J5=-90 exact + FK CAFI error 0.05 mm

Co-Authored-By: Claude Opus 4.7 (1M context) <noreply@anthropic.com>

File: src/schneider_cell_description/urdf/schneider_cell.urdf.xacro (robot description, xacro)
@@ -297,12 +297,16 @@
        z=1.018) so the V36 0.30 m elevated platform is no longer
        needed.  Bins and stations now rest directly on mesa top.   -->
-  <!-- ===== V38 Conveyor (DXF #47: 375 x 150 mm @ DXF 927.5, 775.7) ====
-       World (1.370, 1.365), top-of-belt at z = mesa_top + 0.070 = 1.070.
-       V38 picks on the LEFT side of the belt - notch at local X = -0.135
-       on the south rail, so the rail opening is at world X = 1.235
-       and the cobot grabs from the west (left) end.  Reach to that
-       point from the cobot at (1.252, 1.049) is just 0.353 m.        -->
+  <!-- ===== V57 Conveyor (shifted +0.300 m EAST vs V56) =================
+       Old anchor: (1.370, 1.365), pick at world X = 1.235.
+       New anchor: (1.670, 1.365), pick at world X = 1.535.
+       This is the SECOND +0.30 m shift in the East direction; together
+       with the V56 disc shift the LOAD seat and the conveyor pick are
+       both within a comfortable cobot reach radius, and locking
+       J6_PLACE_LOAD == J6_PICK_CONVEYOR finally becomes feasible.
+       Mesa span: x in [0.442, 2.062], y in [0.589, 1.509].
+       New conveyor span: x in [1.483, 1.858], y in [1.290, 1.440] —
+       still inside mesa with > 200 mm clearance to the east edge.   -->
   <xacro:conveyor_section name="conveyor_1" parent="world"
-                          xy_x="1.370" xy_y="1.365"
+                          xy_x="1.670" xy_y="1.365"
                           size_x="0.375"  size_y="0.150"
                           top_z="1.070"  body_height="0.065"
@@ -311,6 +315,5 @@
                           notch_n_x_local="-0.135"
                           notch_n_w="0.060"/>
-  <!-- ===== V38 Suministro CAFI (feeder at EAST end of belt; CAFIs are
-       fed in from the east and travel west to the left-side pick).  -->
+  <!-- ===== V57 Suministro CAFI (shifted +0.300 m EAST with conveyor) -->
   <link name="suministro_cafi">
     <visual>
@@ -323,5 +326,5 @@
     <parent link="world"/>
     <child  link="suministro_cafi"/>
-    <origin xyz="1.620 1.365 1.0075" rpy="0 0 0"/>
+    <origin xyz="1.920 1.365 1.0075" rpy="0 0 0"/>
   </joint>
   <!-- ===== Quality bins (preserved) ================================== -->
@@ -723,5 +726,5 @@
        NORTH across the belt right at the pick X.                      -->
   <xacro:sick_photoelectric name="sensor_conveyor_end" parent="world"
-                            face_x="1.235" face_y="1.290" face_z="1.100"
+                            face_x="1.535" face_y="1.290" face_z="1.100"
                             beam_yaw="1.5707963267948966"
                             mesa_z="1.000" beam_len="0.150"/>
@@ -742,5 +745,5 @@
   <!-- Conveyor drive motor under EAST end of belt (V38 pick is on west). -->
   <xacro:conveyor_drive_motor name="conveyor_drive_motor" parent="world"
-                              xy_x="1.550" xy_y="1.365" z="1.036"
+                              xy_x="1.850" xy_y="1.365" z="1.036"
                               axis_yaw="1.5707963267948966"/>
   <!-- V41: rotary_drive macro REMOVED.  V37/V38 installed a NEMA-17 +
