Commit message: V61: integrate URDF DEFINITIVO V26 + 2 max-CAFI stress tests
- Add lexium_cobot_v26.urdf (link3_elbow_connector extracted as
  independent link, rpy=(0,pi,0) on joint_elbow_connector) tal cual
  in lexium_cobot_with_final_gripper/urdf, plus display_v26.launch
  to view it in RViz. Kinematics .xacro untouched so the simulation
  keeps its V60 IK and poses.
- Add turntable_rivet_cell_description V11 package (URDF, xacro,
  meshes, launch+rviz) — was only in local v60_ws, now versioned.
- Add v61_max_cafi_test.py with two stress configurations:
    TEST A: 200 CAFIs @5s, alternating PASS/FAIL
    TEST B: 400 CAFIs (100 @4s burst + 300 @5s steady), 267 PASS
            + 133 FAIL
  Both end with cell still RUNNING, 0 faults, 0 watchdogs.
- Re-run resolve_poses.py (19/19 PASS, cart err <= 0.10 mm),
  v56_geom_test (FK err 0.04 mm), v57_collision_test (0 violations
  >=3 cm safety to every plant obstacle).
- Capture all gate logs in evidence/v61/.
- Sync schneider_visualization, rotary_fixture_sim and pose
  collision checker from v60_ws.

File: src/lexium_cobot_with_final_gripper/urdf/lexium_cobot_with_final_gripper.xacro (robot description, xacro)
@@ -134,34 +134,6 @@
     </joint>
     <link name="${name}_gripper_base"/>
-    <!-- visual-only stump marker (centre of mounting plate) -->
-    <link name="${name}_stump_center_marker_link">
-      <visual>
-        <origin xyz="0 0 0" rpy="0 0 0"/>
-        <geometry><sphere radius="0.004"/></geometry>
-        <material name="${name}_mount_center_green">
-          <color rgba="0.0 1.0 0.0 0.85"/>
-        </material>
-      </visual>
-    </link>
-    <joint name="${name}_stump_center_marker_fixed_joint" type="fixed">
-      <parent link="${name}_gripper_base"/>
-      <child  link="${name}_stump_center_marker_link"/>
-      <origin xyz="0 0 0" rpy="0 0 0"/>
-    </joint>
-    <!-- visual-only Z axis reference (open/close direction) -->
-    <link name="${name}_z_axis_reference_link">
-      <visual>
-        <origin xyz="0 0 0.06" rpy="0 0 0"/>
-        <geometry><cylinder radius="0.0015" length="0.12"/></geometry>
-        <material name="${name}_z_axis_blue">
-          <color rgba="0.0 0.25 1.0 0.75"/>
-        </material>
-      </visual>
-    </link>
-    <joint name="${name}_z_axis_reference_fixed_joint" type="fixed">
-      <parent link="${name}_gripper_base"/>
-      <child  link="${name}_z_axis_reference_link"/>
-      <origin xyz="0 0 0" rpy="0 0 0"/>
-    </joint>
+    <!-- V52: stump_center_marker debug sphere REMOVED (visual clutter). -->
+    <!-- V52: z_axis_reference debug cylinder REMOVED (visual clutter). -->
     <!-- stump (mounting plate) -->
     <link name="${name}_stump_link">
@@ -302,33 +274,11 @@
       <origin xyz="0 0 0" rpy="0 0 0"/>
     </joint>
-    <!-- V43 visible TCP marker: 6 mm green sphere at tcp_grasp_center so
-         the user can confirm where the system thinks the TCP is. -->
-    <link name="${name}_tcp_marker_link">
-      <visual>
-        <origin xyz="0 0 0" rpy="0 0 0"/>
-        <geometry><sphere radius="0.006"/></geometry>
-        <material name="${name}_tcp_marker_green">
-          <color rgba="0.10 1.00 0.10 0.95"/>
-        </material>
-      </visual>
-    </link>
-    <joint name="${name}_tcp_marker_fixed_joint" type="fixed">
-      <parent link="${name}_tcp_grasp_center"/>
-      <child  link="${name}_tcp_marker_link"/>
-      <origin xyz="0 0 0" rpy="0 0 0"/>
-    </joint>
-    <!-- V51 golden-reference grasp frames (RViz-only, from the user's
-         debug URDF).  These DO NOT change kinematics; they make the
-         expected CAFI grasp pose visible in RViz so the runtime can
-         be checked against the golden reference. -->
-    <link name="${name}_gripper_grasp_center_frame">
-      <visual>
-        <origin xyz="0 0 0" rpy="0 0 0"/>
-        <geometry><sphere radius="0.006"/></geometry>
-        <material name="${name}_grasp_center_yellow">
-          <color rgba="1.0 0.9 0.0 0.85"/>
-        </material>
-      </visual>
-    </link>
+    <!-- V52 visual cleanup: debug spheres / boxes removed.  The frames
+         themselves are kept as EMPTY links because robot_controller,
+         pose resolver and object_manager address them by name; only the
+         visual tags are dropped so RViz no longer shows the debug helpers
+         (transparent cyan grasp box, yellow contact spheres, green TCP
+         dot, yellow grasp-center dot). -->
+    <link name="${name}_gripper_grasp_center_frame"/>
     <joint name="${name}_gripper_grasp_center_fixed_joint" type="fixed">
       <parent link="${name}_gripper_base"/>
@@ -336,13 +286,5 @@
       <origin xyz="0.000000 0.016600 0.076750" rpy="0 0 0"/>
     </joint>
-    <link name="${name}_appendage_inner_contact_frame">
-      <visual>
-        <origin xyz="0 0 0" rpy="0 0 0"/>
-        <geometry><sphere radius="0.0045"/></geometry>
-        <material name="${name}_appendage_inner_yellow">
-          <color rgba="1.0 0.9 0.0 0.85"/>
-        </material>
-      </visual>
-    </link>
+    <link name="${name}_appendage_inner_contact_frame"/>
     <joint name="${name}_appendage_inner_contact_fixed_joint" type="fixed">
       <parent link="${name}_appendage_link"/>
@@ -350,13 +292,5 @@
       <origin xyz="0.000250 0.060250 0.076750" rpy="0 0 0"/>
     </joint>
-    <link name="${name}_fixed_jaw_inner_contact_frame">
-      <visual>
-        <origin xyz="0 0 0" rpy="0 0 0"/>
-        <geometry><sphere radius="0.0045"/></geometry>
-        <material name="${name}_fixed_jaw_yellow">
-          <color rgba="1.0 0.9 0.0 0.85"/>
-        </material>
-      </visual>
-    </link>
+    <link name="${name}_fixed_jaw_inner_contact_frame"/>
     <joint name="${name}_fixed_jaw_inner_contact_fixed_joint" type="fixed">
       <parent link="${name}_gripper_base"/>
@@ -364,13 +298,5 @@
       <origin xyz="0.000000 -0.027050 0.076750" rpy="0 0 0"/>
     </joint>
-    <link name="${name}_cafi_lateral_target_frame">
-      <visual>
-        <origin xyz="0 0 0" rpy="0 0 0"/>
-        <geometry><sphere radius="0.0055"/></geometry>
-        <material name="${name}_cafi_target_green">
-          <color rgba="0.0 1.0 0.0 0.85"/>
-        </material>
-      </visual>
-    </link>
+    <link name="${name}_cafi_lateral_target_frame"/>
     <joint name="${name}_cafi_lateral_target_fixed_joint" type="fixed">
       <parent link="${name}_gripper_base"/>
@@ -378,13 +304,5 @@
       <origin xyz="0.000000 0.016600 0.076750" rpy="0 0 0"/>
     </joint>
-    <link name="${name}_grasp_volume_frame">
-      <visual>
-        <origin xyz="0 0 0" rpy="0 0 0"/>
-        <geometry><box size="0.126 0.090 0.030"/></geometry>
-        <material name="${name}_grasp_volume_cyan">
-          <color rgba="0.1 0.8 1.0 0.25"/>
-        </material>
-      </visual>
-    </link>
+    <link name="${name}_grasp_volume_frame"/>
     <joint name="${name}_grasp_volume_fixed_joint" type="fixed">
       <parent link="${name}_cafi_lateral_target_frame"/>
