Commit message: Update simulation to V51
Core change: replace scalar LATERAL_GRASP_OFFSET and ad-hoc
PICK_CONVEYOR_TARGET_DX_WORLD with vector LATERAL_GRASP_DELTA extracted
byte-for-byte from the gripper URDF debug golden reference. New IK
formula: TCP_world = CAFI_world + R_gripper_world * LATERAL_GRASP_DELTA.

Adds debug-only frames to gripper URDF (cafi_lateral_target_frame,
gripper_grasp_center_frame, appendage_inner_contact_frame, etc.) —
visual only, kinematics unchanged.

Includes V50 and V51 cycle/IK/collision evidence and expanded URDFs,
plus full V51 design notes in schneider_cell_description_V51_resumen.md.

File: src/lexium_cobot_with_final_gripper/urdf/lexium_cobot_with_final_gripper.urdf (robot description, URDF)
Before this commit: robot lexium_cobot_with_final_gripper, 18 links, 17 joints
Links:
- added link appendage_inner_contact_frame; visual sphere radius=0.0045
- added link cafi_lateral_target_frame; visual sphere radius=0.0055
- added link fixed_jaw_inner_contact_frame; visual sphere radius=0.0045
- added link grasp_volume_frame; visual box size=0.126 0.090 0.030
- added link gripper_grasp_center_frame; visual sphere radius=0.006
Joints:
- added joint appendage_inner_contact_fixed_joint: type fixed, parent appendage_link, child appendage_inner_contact_frame, origin xyz=0.000250 0.060250 0.076750 rpy=0 0 0
- added joint cafi_lateral_target_fixed_joint: type fixed, parent gripper_base, child cafi_lateral_target_frame, origin xyz=0.000000 0.016600 0.076750 rpy=0 0 0
- added joint fixed_jaw_inner_contact_fixed_joint: type fixed, parent gripper_base, child fixed_jaw_inner_contact_frame, origin xyz=0.000000 -0.027050 0.076750 rpy=0 0 0
- added joint grasp_volume_fixed_joint: type fixed, parent cafi_lateral_target_frame, child grasp_volume_frame, origin xyz=0 0 0 rpy=0 0 0
- added joint gripper_grasp_center_fixed_joint: type fixed, parent gripper_base, child gripper_grasp_center_frame, origin xyz=0.000000 0.016600 0.076750 rpy=0 0 0

File: src/lexium_cobot_with_final_gripper/urdf/lexium_cobot_with_final_gripper.xacro (robot description, xacro)
@@ -318,4 +318,78 @@
       <origin xyz="0 0 0" rpy="0 0 0"/>
     </joint>
+    <!-- V51 golden-reference grasp frames (RViz-only, from the user's
+         debug URDF).  These DO NOT change kinematics; they make the
+         expected CAFI grasp pose visible in RViz so the runtime can
+         be checked against the golden reference. -->
+    <link name="${name}_gripper_grasp_center_frame">
+      <visual>
+        <origin xyz="0 0 0" rpy="0 0 0"/>
+        <geometry><sphere radius="0.006"/></geometry>
+        <material name="${name}_grasp_center_yellow">
+          <color rgba="1.0 0.9 0.0 0.85"/>
+        </material>
+      </visual>
+    </link>
+    <joint name="${name}_gripper_grasp_center_fixed_joint" type="fixed">
+      <parent link="${name}_gripper_base"/>
+      <child  link="${name}_gripper_grasp_center_frame"/>
+      <origin xyz="0.000000 0.016600 0.076750" rpy="0 0 0"/>
+    </joint>
+    <link name="${name}_appendage_inner_contact_frame">
+      <visual>
+        <origin xyz="0 0 0" rpy="0 0 0"/>
+        <geometry><sphere radius="0.0045"/></geometry>
+        <material name="${name}_appendage_inner_yellow">
+          <color rgba="1.0 0.9 0.0 0.85"/>
+        </material>
+      </visual>
+    </link>
+    <joint name="${name}_appendage_inner_contact_fixed_joint" type="fixed">
+      <parent link="${name}_appendage_link"/>
+      <child  link="${name}_appendage_inner_contact_frame"/>
+      <origin xyz="0.000250 0.060250 0.076750" rpy="0 0 0"/>
+    </joint>
+    <link name="${name}_fixed_jaw_inner_contact_frame">
+      <visual>
+        <origin xyz="0 0 0" rpy="0 0 0"/>
+        <geometry><sphere radius="0.0045"/></geometry>
+        <material name="${name}_fixed_jaw_yellow">
+          <color rgba="1.0 0.9 0.0 0.85"/>
+        </material>
+      </visual>
+    </link>
+    <joint name="${name}_fixed_jaw_inner_contact_fixed_joint" type="fixed">
+      <parent link="${name}_gripper_base"/>
+      <child  link="${name}_fixed_jaw_inner_contact_frame"/>
+      <origin xyz="0.000000 -0.027050 0.076750" rpy="0 0 0"/>
+    </joint>
+    <link name="${name}_cafi_lateral_target_frame">
+      <visual>
+        <origin xyz="0 0 0" rpy="0 0 0"/>
+        <geometry><sphere radius="0.0055"/></geometry>
+        <material name="${name}_cafi_target_green">
+          <color rgba="0.0 1.0 0.0 0.85"/>
+        </material>
+      </visual>
+    </link>
+    <joint name="${name}_cafi_lateral_target_fixed_joint" type="fixed">
+      <parent link="${name}_gripper_base"/>
+      <child  link="${name}_cafi_lateral_target_frame"/>
+      <origin xyz="0.000000 0.016600 0.076750" rpy="0 0 0"/>
+    </joint>
+    <link name="${name}_grasp_volume_frame">
+      <visual>
+        <origin xyz="0 0 0" rpy="0 0 0"/>
+        <geometry><box size="0.126 0.090 0.030"/></geometry>
+        <material name="${name}_grasp_volume_cyan">
+          <color rgba="0.1 0.8 1.0 0.25"/>
+        </material>
+      </visual>
+    </link>
+    <joint name="${name}_grasp_volume_fixed_joint" type="fixed">
+      <parent link="${name}_cafi_lateral_target_frame"/>
+      <child  link="${name}_grasp_volume_frame"/>
+      <origin xyz="0 0 0" rpy="0 0 0"/>
+    </joint>
   </xacro:macro>
 </robot>

Commit message: V61: swap cobot URDF in-place for URDF DEFINITIVO
Reemplaza literalmente el cobot que estaba en la simulacion por el
URDF DEFINITIVO provisto en URDF_DEFINITIVO.zip:

  src/lexium_cobot_with_final_gripper/urdf/lexium_cobot_with_final_gripper.urdf
  src/lexium_cobot_with_final_gripper/urdf/lexium_cobot_with_final_gripper.xacro

Cinematica: link3_elbow_connector ahora es link independiente, con
joint_elbow_connector (fixed, rpy=(0,pi,0)) heredando la rotacion 180Y
concentrica del pivot.  joint_3 y la cadena subsecuente cuelgan de
link_elbow_connector.  Visual origins de links downstream identicos
al URDF definitivo original.

Mesh filenames del .urdf usan package:// para que cargue desde
cualquier launch ROS.  El .xacro preserva el macro
lexium_cobot_with_final_gripper(name, parent, mount_xyz, mount_rpy) y
el alias ${name}_tcp_grasp_center que el resto del sim direcciona por
nombre.

Removidos por redundancia con esta swap:
  src/lexium_cobot_with_final_gripper/urdf/lexium_cobot_v26.urdf
  src/lexium_cobot_with_final_gripper/launch/display_v26.launch

File: src/lexium_cobot_with_final_gripper/urdf/lexium_cobot_with_final_gripper.urdf (robot description, URDF)
Before this commit: robot lexium_cobot_with_final_gripper, 23 links, 22 joints
Links:
- removed link appendage_inner_contact_frame
- removed link fixed_jaw_inner_contact_frame
- removed link grasp_volume_frame
- removed link gripper_grasp_center_frame
- removed link stump_center_marker_link
- removed link z_axis_reference_link
- added link link_elbow_connector; visual mesh filename=package://lexium_cobot_with_final_gripper/meshes/cobot/link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 scale=0.001 0.001 0.001
- link appendage_link: geometry visual mesh filename=package://lexium_cobot_with_final_gripper/meshes/gripper/ap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 scale=0.001 0.001 0.001
- link base_link: mass 3.5 -> None; geometry visual mesh filename=package://lexium_cobot_with_final_gripper/meshes/cobot/link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 scale=0.001 0.001 0.001
- link cafi_lateral_target_frame: geometry 
- link fixture1_link: geometry visual mesh filename=package://lexium_cobot_with_final_gripper/meshes/gripper/fi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 scale=0.001 0.001 0.001
- link fixture_link: geometry visual mesh filename=package://lexium_cobot_with_final_gripper/meshes/gripper/fi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 scale=0.001 0.001 0.001
- link link1_shoulder: mass 2.0 -> None; geometry visual mesh filename=package://lexium_cobot_with_final_gripper/meshes/cobot/link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 scale=0.001 0.001 0.001
- link link2_upper_arm: mass 1.8 -> None; geometry visual mesh filename=package://lexium_cobot_with_final_gripper/meshes/cobot/link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 scale=0.001 0.001 0.001; visual mesh filename=package://lexium_cobot_with_final_gripper/meshes/cobot/link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 scale=0.001 0.001 0.001
- link link3_forearm: mass 1.2 -> None; geometry visual mesh filename=package://lexium_cobot_with_final_gripper/meshes/cobot/link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 scale=0.001 0.001 0.001; visual mesh filename=package://lexium_cobot_with_final_gripper/meshes/cobot/link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 scale=0.001 0.001 0.001
- link link4_wrist1: mass 0.8 -> None; geometry visual mesh filename=package://lexium_cobot_with_final_gripper/meshes/cobot/link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 scale=0.001 0.001 0.001; visual mesh filename=package://lexium_cobot_with_final_gripper/meshes/cobot/link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 scale=0.001 0.001 0.001
- link link5_wrist2: mass 0.4 -> None; geometry visual mesh filename=package://lexium_cobot_with_final_gripper/meshes/cobot/link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 scale=0.001 0.001 0.001
- link link6_wrist3: mass 0.3 -> None; geometry visual mesh filename=package://lexium_cobot_with_final_gripper/meshes/cobot/link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 scale=0.001 0.001 0.001
- link neck_link: geometry visual mesh filename=package://lexium_cobot_with_final_gripper/meshes/gripper/ne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 scale=0.001 0.001 0.001
- link stump_link: geometry visual mesh filename=package://lexium_cobot_with_final_gripper/meshes/gripper/st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 scale=0.001 0.001 0.001
Joints:
- removed joint appendage_inner_contact_fixed_joint
- removed joint fixed_jaw_inner_contact_fixed_joint
- removed joint grasp_volume_fixed_joint
- removed joint gripper_grasp_center_fixed_joint
- removed joint stump_center_marker_fixed_joint
- removed joint z_axis_reference_fixed_joint
- added joint joint_elbow_connector: type fixed, parent link2_upper_arm, child link_elbow_connector, origin xyz=0.001060 0.243625 0.119967 rpy=0 3.14159265359 0
- joint joint_1: limit lower=-3.14159 upper=3.14159 effort=50.0 velocity=3.14 -> lower=-3.14159 upper=3.14159 effort=50 velocity=3.14
- joint joint_2: limit lower=-2.61799 upper=2.61799 effort=50.0 velocity=3.14 -> lower=-2.61799 upper=2.61799 effort=50 velocity=3.14; origin xyz=-0.0115 0.0639 0.0000 rpy=0 0 0.05 -> xyz=-0.0115 0.0639 0 rpy=0 0 0.05
- joint joint_3: limit lower=-2.61799 upper=2.61799 effort=50.0 velocity=3.14 -> lower=-2.61799 upper=2.61799 effort=50 velocity=3.14; origin xyz=-0.0015 0.2450 0.2258 rpy=0 0 0 -> xyz=0.002560 0.001375 0.113592 rpy=0 0 0; parent link2_upper_arm -> link_elbow_connector
- joint joint_4: limit lower=-3.14159 upper=3.14159 effort=50.0 velocity=3.14 -> lower=-3.14159 upper=3.14159 effort=50 velocity=3.14
- joint joint_5: limit lower=-2.09440 upper=2.09440 effort=50.0 velocity=3.14 -> lower=-2.09440 upper=2.09440 effort=50 velocity=3.14
- joint joint_6: limit lower=-3.14159 upper=3.14159 effort=50.0 velocity=3.14 -> lower=-3.14159 upper=3.14159 effort=50 velocity=3.14
- joint tool0_to_gripper_base: origin xyz=0.0 -0.07 0.015 rpy=0 0 0 -> xyz=0 -0.07 0.015 rpy=0 0 0
